File: PCB/Pi Hat/Pi Hat.kicad_pcb (KiCad board)
At the start: 2 copper layers, 26.7 x 55.9 mm, 11 parts, among them IC1 MCP3008-I_SL, J1 Conn_01x04, J2 Conn_02x20_Odd_Even, J3 Conn_01x03, J4 Conn_01x02, U1 74LVC2T45DC

Commit message: completed PCB
Parts:
- added TP1: TestPoint, TestPoint:TestPoint_Pad_D3.0mm, F.Cu at (105.2, 75.6)
- added TP2: TestPoint, TestPoint:TestPoint_Pad_D3.0mm, F.Cu at (94.0, 59.8)
- added TP3: TestPoint, TestPoint:TestPoint_Pad_D3.0mm, F.Cu at (107.8, 111.0)
Routing:
- net /ForceVoltage: track 24.3 -> 29.1 mm
- net +5V: track 40.3 -> 41.9 mm
- net +3.3V: track 116.0 -> 116.7 mm
- net GND: vias 2 -> 3
Other:
- board text added: "DH11"
- board text added: "FSR"
- board text added: "HC-SR04"
