File: PCB/Pi Hat/Pi Hat.kicad_pcb (KiCad board)
At the start: 2 copper layers, 26.7 x 55.9 mm, 14 parts, among them IC1 MCP3008-I_SL, J1 Conn_01x04, J2 Conn_02x20_Odd_Even, J3 Conn_01x03, J4 Conn_01x02, U1 74LVC2T45DC

Commit message: complete PCB
Parts:
- added J5: Conn_01x03, Connector_Molex:Molex_KK-254_AE-6410-03A_1x03_P2.54mm_Vertical, F.Cu at (177.8, 96.5)
- moved TP3 113.4 mm to (208.3, 58.4), turned to 90 degrees
- moved R1 101.9 mm to (204.1, 81.3)
- moved IC1 99.1 mm to (198.1, 81.3), turned to 180 degrees
- moved J4 97.4 mm to (195.6, 96.5), turned to 180 degrees
- moved TP2 91.4 mm to (182.9, 81.3)
- moved J3 90.2 mm to (188.0, 96.5), turned to 180 degrees
- moved D1 86.3 mm to (186.4, 88.9), turned to 0 degrees
- moved R2 84.5 mm to (186.3, 86.4), turned to 0 degrees
- moved J1 73.1 mm to (167.6, 96.5), turned to 180 degrees
- moved U1 59.9 mm to (165.1, 83.8), turned to -90 degrees
- moved TP1 46.1 mm to (151.1, 71.1), turned to -90 degrees
- moved D2 45.7 mm to (152.1, 63.5), turned to 0 degrees
- moved R3 45.6 mm to (152.0, 66.0), turned to 0 degrees
- moved J2 44.2 mm to (154.9, 51.3), turned to -90 degrees
Connections:
- J2 pad 12: unconnected-(J2-Pin_12-Pad12) -> /PWM_0
- J4 pad 1: +3.3V -> /ForceVoltage
- J4 pad 2: /ForceVoltage -> +3.3V
Routing:
- net +5V: track 41.9 -> 120.9 mm, vias 2 -> 1
- net /PWM_0: track 0.00 -> 54.5 mm
- net /Data_3.3VTTL: track 12.7 -> 50.5 mm
- net /Trigger_3.3VTTL: track 4.79 -> 31.9 mm
- net /Echo_3.3VTTL: track 9.25 -> 35.9 mm, vias 0 -> 2
- net /ConverterDir: track 11.4 -> 37.9 mm, vias 1 -> 0
- net /SCLK: track 6.65 -> 28.5 mm, vias 0 -> 1
- net +3.3V: track 116.7 -> 100.3 mm, vias 0 -> 2
- net /CS: track 6.65 -> 16.9 mm
- net /MISO: track 14.6 -> 24.1 mm
- net /ForceVoltage: track 29.1 -> 21.4 mm
- net /MOSI: track 21.2 -> 28.5 mm, vias 0 -> 1
- net /Trigger_5VTTL: track 6.91 -> 11.3 mm
- net /Echo_5VTTL: track 7.76 -> 12.1 mm
- net GND: track 2.20 -> 1.21 mm, vias 3 -> 1
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Other:
- board size 26.7 x 55.9 mm -> 68 x 59 mm
- board text added: "SERVO"

Commit message: DFM check adjustments
Routing:
- net GND: track 1.21 -> 1.78 mm
Changed lines of the file:
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@@
   )
   (setup
+    (stackup
+      (layer "F.SilkS" (type "Top Silk Screen"))
+      (layer "F.Paste" (type "Top Solder Paste"))
+      (layer "F.Mask" (type "Top Solder Mask") (thickness 0.01))
+      (layer "F.Cu" (type "copper") (thickness 0.035))
+      (layer "dielectric 1" (type "core") (thickness 1.51) (material "FR4") (epsilon_r 4.5) (loss_tangent 0.02))
+      (layer "B.Cu" (type "copper") (thickness 0.035))
+      (layer "B.Mask" (type "Bottom Solder Mask") (thickness 0.01))
+      (layer "B.Paste" (type "Bottom Solder Paste"))
+      (layer "B.SilkS" (type "Bottom Silk Screen"))
+      (copper_finish "None")
+      (dielectric_constraints no)
+    )
     (pad_to_mask_clearance 0)
     (grid_origin 180.34 86.36)
@@
     (property "ki_keywords" "R res resistor")
     (attr smd)
-    (fp_text reference "R3" (at 0 -2.174 90) (layer "F.SilkS")
+    (fp_text reference "R3" (at -3.4525 -2.54 180) (layer "F.SilkS")
         (effects (font (size 1 1) (thickness 0.15)))
     )
@@
     (fp_line (start 6.35 2.88) (end 6.35 -2.92)
       (stroke (width 0.1) (type solid)) (layer "F.Fab"))
-    (pad "1" thru_hole roundrect (at 0 0 180) (size 1.74 2.19) (drill 1.19) (layers "*.Cu" "*.Mask") (roundrect_rratio 0.143678)
+    (pad "1" thru_hole roundrect (at 0 0 180) (size 1.74 2.19) (drill 1.19) (layers "*.Cu" "*.Mask") (roundrect_rratio 0.1436781609)
       (net 1 "+5V") (pinfunction "Pin_1") (pintype "passive"))
     (pad "2" thru_hole oval (at 2.54 0 180) (size 1.74 2.19) (drill 1.19) (layers "*.Cu" "*.Mask")
@@
     (property "ki_keywords" "R res resistor")
     (attr smd)
-    (fp_text reference "R2" (at 2.5525 0.921 90) (layer "F.SilkS")
+    (fp_text reference "R2" (at -3.4525 0 180) (layer "F.SilkS")
         (effects (font (size 1 1) (thickness 0.15)))
     )
@@
     (property "ki_keywords" "LED diode")
     (attr smd)
-    (fp_text reference "D1" (at 1.0435 -1.921 90) (layer "F.SilkS")
+    (fp_text reference "D1" (at -3.4775 0 180) (layer "F.SilkS")
         (effects (font (size 1 1) (thickness 0.15)))
     )
@@
     (property "ki_keywords" "LED diode")
     (attr smd)
-    (fp_text reference "D2" (at 0 2.174 90) (layer "F.SilkS")
+    (fp_text reference "D2" (at -3.4775 2.54 180) (layer "F.SilkS")
         (effects (font (size 1 1) (thickness 0.15)))
     )
@@
   (segment (start 152.4 50.047919) (end 152.4 55.88) (width 1) (layer "B.Cu") (net 2))
   (segment (start 152.4 55.88) (end 167.64 71.12) (width 1) (layer "B.Cu") (net 2))
-  (segment (start 164.35 81.8) (end 163.83 81.28) (width 0.3) (layer "F.Cu") (net 5))
-  (segment (start 164.35 82.27) (end 164.35 81.8) (width 0.3) (layer "F.Cu") (net 5))
-  (via (at 163.83 81.28) (size 0.4) (drill 0.2) (layers "F.Cu" "B.Cu") (net 5))
-  (segment (start 165.35 82.27) (end 165.35 53.54) (width 0.3) (layer "F.Cu") (net 8))
-  (segment (start 165.35 53.54) (end 167.6 51.29) (width 0.3) (layer "F.Cu") (net 8))
+  (segment (start 164.35 81.083034) (end 163.933259 80.666293) (width 0.3) (layer "F.Cu") (net 5))
+  (segment (start 164.35 82.27) (end 164.35 81.083034) (width 0.3) (layer "F.Cu") (net 5))
+  (via (at 163.933259 80.666293) (size 0.6) (drill 0.3) (layers "F.Cu" "B.Cu") (net 5))
+  (segment (start 165.872921 81.116437) (end 165.872921 53.017079) (width 0.3) (layer "F.Cu") (net 8))
+  (segment (start 165.35 82.27) (end 165.35 81.639358) (width 0.3) (layer "F.Cu") (net 8))
+  (segment (start 165.35 81.639358) (end 165.872921 81.116437) (width 0.3) (layer "F.Cu") (net 8))
+  (segment (start 165.872921 53.017079) (end 167.6 51.29) (width 0.3) (layer "F.Cu") (net 8))
   (segment (start 171.48 48.29) (end 171.48 92.74) (width 0.3) (layer "F.Cu") (net 9))
   (segment (start 171.48 92.74) (end 175.26 96.52) (width 0.3) (layer "F.Cu") (net 9))
@@
   (segment (start 170.74 47.55) (end 171.48 48.29) (width 0.3) (layer "F.Cu") (net 9))
   (segment (start 167.6 48.75) (end 168.8 47.55) (width 0.3) (layer "F.Cu") (net 9))
+  (segment (start 164.906714 79.512923) (end 164.133791 78.74) (width 0.3) (layer "F.Cu") (net 10))
+  (segment (start 164.85 82.27) (end 164.85 81.432252) (width 0.3) (layer "F.Cu") (net 10))
   (segment (start 170.14 51.29) (end 167.005 54.425) (width 0.3) (layer "F.Cu") (net 10))
-  (segment (start 164.85 79.76) (end 163.83 78.74) (width 0.3) (layer "F.Cu") (net 10))
+  (segment (start 164.85 81.432252) (end 164.906714 81.375538) (width 0.3) (layer "F.Cu") (net 10))
   (segment (start 167.005 54.425) (end 167.005 78.74) (width 0.3) (layer "F.Cu") (net 10))
-  (segment (start 164.85 82.27) (end 164.85 79.76) (width 0.3) (layer "F.Cu") (net 10))
-  (via (at 163.83 78.74) (size 0.4) (drill 0.2) (layers "F.Cu" "B.Cu") (net 10))
-  (via (at 167.005 78.74) (size 0.4) (drill 0.2) (layers "F.Cu" "B.Cu") (net 10))
-  (segment (start 167.005 78.74) (end 163.83 78.74) (width 0.3) (layer "B.Cu") (net 10))
+  (segment (start 164.906714 81.375538) (end 164.906714 79.512923) (width 0.3) (layer "F.Cu") (net 10))
+  (via (at 164.133791 78.74) (size 0.6) (drill 0.3) (layers "F.Cu" "B.Cu") (net 10))
+  (via (at 167.005 78.74) (size 0.6) (drill 0.3) (layers "F.Cu" "B.Cu") (net 10))
+  (segment (start 167.005 78.74) (end 164.133791 78.74) (width 0.3) (layer "B.Cu") (net 10))
   (segment (start 172.68 51.29) (end 172.68 83.78) (width 1) (layer "F.Cu") (net 11))
   (segment (start 172.68 83.78) (end 185.42 96.52) (width 1) (layer "F.Cu") (net 11))
-  (segment (start 163.2 84.22) (end 163.2 52.7) (width 0.3) (layer "F.Cu") (net 17))
+  (segment (start 163.83 50.06) (end 162.52 48.75) (width 0.3) (layer "F.Cu") (net 17))
+  (segment (start 163.014496 52.885504) (end 163.83 52.07) (width 0.3) (layer "F.Cu") (net 17))
+  (segment (start 164.35 85.37) (end 163.014496 84.034496) (width 0.3) (layer "F.Cu") (net 17))
+  (segment (start 163.014496 84.034496) (end 163.014496 52.885504) (width 0.3) (layer "F.Cu") (net 17))
   (segment (start 163.83 52.07) (end 163.83 50.06) (width 0.3) (layer "F.Cu") (net 17))
-  (segment (start 163.2 52.7) (end 163.83 52.07) (width 0.3) (layer "F.Cu") (net 17))
-  (segment (start 164.35 85.37) (end 163.2 84.22) (width 0.3) (layer "F.Cu") (net 17))
-  (segment (start 163.83 50.06) (end 162.52 48.75) (width 0.3) (layer "F.Cu") (net 17))
   (segment (start 164.85 85.37) (end 164.85 94.23) (width 0.3) (layer "F.Cu") (net 27))
   (segment (start 164.85 94.23) (end 162.56 96.52) (width 0.3) (layer "F.Cu") (net 27))
