File: PCB/Pi Hat/Pi Hat.kicad_sch (KiCad schematic)
At the start: 11 parts, among them IC1 MCP3008-I_SL, J1 Conn_01x04, J2 Conn_02x20_Odd_Even, J3 Conn_01x03, J4 Conn_01x02, U1 74LVC2T45DC

Commit message: completed PCB
Parts:
- added TP1, TP2, TP3: TestPoint, TestPoint:TestPoint_Pad_D3.0mm, symbol Connector:TestPoint
Connections:
- net +3.3V: now also TP2.1
- net +5V: now also TP1.1
- net GND: now also TP3.1
Changed lines of the file:
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@@
   (junction (at 129.54 99.06) (diameter 0) (color 0 0 0 0)
+  )
+  (junction (at 129.54 139.7) (diameter 0) (color 0 0 0 0)
   )
   (junction (at 198.12 63.5) (diameter 0) (color 0 0 0 0)
@@
     (stroke (width 0) (type default))
   )
+  (wire (pts (xy 137.16 83.82) (xy 149.86 83.82))
+    (stroke (width 0) (type default))
+  )
   (wire (pts (xy 88.9 106.68) (xy 114.3 106.68))
     (stroke (width 0) (type default))
@@
   )
   (wire (pts (xy 38.1 55.88) (xy 38.1 58.42))
+    (stroke (width 0) (type default))
+  )
+  (wire (pts (xy 88.9 83.82) (xy 104.14 83.82))
     (stroke (width 0) (type default))
   )
@@
         (path "/2837f593-2859-4fb0-9481-b616afb06594"
           (reference "R3") (unit 1)
+        )
+      )
+    )
+  )
+  (symbol (lib_id "Connector:TestPoint") (at 149.86 83.82 0) (mirror y) (unit 1)
+    (in_bom yes) (on_board yes) (dnp no)
+    (property "Reference" "TP2" (at 152.4 79.248 0)
+      (effects (font (size 1.27 1.27)) (justify right))
+    )
+    (property "Value" "TestPoint" (at 152.4 81.788 0)
+      (effects (font (size 1.27 1.27)) (justify right))
+    )
+    (property "Footprint" "TestPoint:TestPoint_Pad_D3.0mm" (at 144.78 83.82 0)
+      (effects (font (size 1.27 1.27)) hide)
+    )
+    (property "Datasheet" "~" (at 144.78 83.82 0)
+      (effects (font (size 1.27 1.27)) hide)
+    )
+    (pin "1")
+    (instances
+      (project "Pi Hat"
+        (path "/2837f593-2859-4fb0-9481-b616afb06594"
+          (reference "TP2") (unit 1)
         )
       )
@@
     )
   )
+  (symbol (lib_id "Connector:TestPoint") (at 88.9 83.82 0) (unit 1)
+    (in_bom yes) (on_board yes) (dnp no)
+    (property "Reference" "TP1" (at 86.36 79.248 0)
+      (effects (font (size 1.27 1.27)) (justify right))
+    )
+    (property "Value" "TestPoint" (at 86.36 81.788 0)
+      (effects (font (size 1.27 1.27)) (justify right))
+    )
+    (property "Footprint" "TestPoint:TestPoint_Pad_D3.0mm" (at 93.98 83.82 0)
+      (effects (font (size 1.27 1.27)) hide)
+    )
+    (property "Datasheet" "~" (at 93.98 83.82 0)
+      (effects (font (size 1.27 1.27)) hide)
+    )
+    (pin "1")
+    (instances
+      (project "Pi Hat"
+        (path "/2837f593-2859-4fb0-9481-b616afb06594"
+          (reference "TP1") (unit 1)
+        )
+      )
+    )
+  )
   (symbol (lib_id "power:+3.3V") (at 203.2 114.3 0) (unit 1)
     (in_bom yes) (on_board yes) (dnp no) (fields_autoplaced)
@@
         )
       )
+    )
+  )
+  (symbol (lib_id "Connector:TestPoint") (at 129.54 139.7 180) (unit 1)
+    (in_bom yes) (on_board yes) (dnp no)
+    (property "Reference" "TP3" (at 132.08 144.272 0)
+      (effects (font (size 1.27 1.27)) (justify right))
+    )
+    (property "Value" "TestPoint" (at 132.08 141.732 0)
+      (effects (font (size 1.27 1.27)) (justify right))
+    )
+    (property "Footprint" "TestPoint:TestPoint_Pad_D3.0mm" (at 124.46 139.7 0)
+      (effects (font (size 1.27 1.27)) hide)
+    )
+    (property "Datasheet" "~" (at 124.46 139.7 0)
+      (effects (font (size 1.27 1.27)) hide)
+    )
+    (pin "1")
+    (instances
+      (project "Pi Hat"
+        (path "/2837f593-2859-4fb0-9481-b616afb06594"
+          (reference "TP3") (unit 1)
+        )
+      )

Commit message: complete PCB
Parts:
- added J5: Conn_01x03, Connector_Molex:Molex_KK-254_AE-6410-03A_1x03_P2.54mm_Vertical, symbol Connector_Generic:Conn_01x03
Connections:
- net +3.3V: now also J4.2 (Pin_2); no longer J4.1 (Pin_1)
- net +5V: now also J5.1 (Pin_1)
- net ForceVoltage: now also J4.1 (Pin_1); no longer J4.2 (Pin_2)
- net GND: now also J5.3 (Pin_3)
- net PWM_0: now reaches J2.12 (Pin_12)
- net PWM_0: now also J5.2 (Pin_2)
Other:
- note added: "Servo Output:"
Changed lines of the file:
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@@
   (no_connect (at 127 116.84))
   (no_connect (at 127 104.14))
+  (no_connect (at 114.3 116.84))
   (no_connect (at 236.22 58.42))
   (no_connect (at 127 109.22))
@@
   (no_connect (at 114.3 91.44))
   (no_connect (at 127 101.6))
-  (no_connect (at 127 96.52))
   (no_connect (at 127 114.3))
   (no_connect (at 236.22 55.88))
@@
     (stroke (width 0) (type default))
   )
+  (wire (pts (xy 114.3 180.34) (xy 111.76 180.34))
+    (stroke (width 0) (type default))
+  )
   (wire (pts (xy 205.74 142.24) (xy 205.74 144.78))
     (stroke (width 0) (type default))
@@
     (stroke (width 0) (type default))
   )
+  (wire (pts (xy 152.4 96.52) (xy 127 96.52))
+    (stroke (width 0) (type default))
+  )
   (wire (pts (xy 114.3 93.98) (xy 111.76 93.98))
     (stroke (width 0) (type default))
@@
     (stroke (width 0) (type default))
   )
+  (wire (pts (xy 88.9 177.8) (xy 114.3 177.8))
+    (stroke (width 0) (type default))
+  )
+  (wire (pts (xy 111.76 180.34) (xy 111.76 182.88))
+    (stroke (width 0) (type default))
+  )
   (wire (pts (xy 203.2 48.26) (xy 200.66 48.26))
     (stroke (width 0) (type default))
@@
     (stroke (width 0) (type default))
   )
+  (wire (pts (xy 111.76 172.72) (xy 111.76 175.26))
+    (stroke (width 0) (type default))
+  )
   (wire (pts (xy 38.1 55.88) (xy 38.1 58.42))
     (stroke (width 0) (type default))
@@
   )
   (wire (pts (xy 241.3 40.64) (xy 248.92 40.64))
+    (stroke (width 0) (type default))
+  )
+  (wire (pts (xy 111.76 175.26) (xy 114.3 175.26))
     (stroke (width 0) (type default))
   )
@@
     (fill (type none))
   )
+  (rectangle (start 93.98 157.48) (end 137.16 195.58)
+    (stroke (width 0) (type dash))
+    (fill (type none))
+  )
   (rectangle (start 172.72 17.78) (end 276.86 88.9)
     (stroke (width 0) (type dash))
@@
     (effects (font (size 1.27 1.27)) (justify left bottom))
   )
+  (text "Servo Output:" (at 96.52 162.56 0)
+    (effects (font (size 1.27 1.27)) (justify left bottom))
+  )
   (text "Force Sensitive Resistor" (at 175.26 22.86 0)
     (effects (font (size 1.27 1.27)) (justify left bottom))
@@
     (effects (font (size 1.27 1.27)) (justify right bottom))
   )
+  (label "PWM_0" (at 152.4 96.52 0) (fields_autoplaced)
+    (effects (font (size 1.27 1.27)) (justify left bottom))
+  )
   (label "MOSI" (at 88.9 106.68 180) (fields_autoplaced)
     (effects (font (size 1.27 1.27)) (justify right bottom))
@@
   )
   (label "Echo_3.3VTTL" (at 88.9 99.06 180) (fields_autoplaced)
+    (effects (font (size 1.27 1.27)) (justify right bottom))
+  )
+  (label "PWM_0" (at 88.9 177.8 180) (fields_autoplaced)
     (effects (font (size 1.27 1.27)) (justify right bottom))
   )
@@
     )
   )
-  (symbol (lib_id "Connector_Generic:Conn_01x02") (at 256.54 38.1 0) (unit 1)
-    (in_bom yes) (on_board yes) (dnp no) (fields_autoplaced)
-    (property "Reference" "J4" (at 259.08 38.1 0)
+  (symbol (lib_id "power:GND") (at 111.76 182.88 0) (unit 1)
+    (in_bom yes) (on_board yes) (dnp no) (fields_autoplaced)
+    (property "Reference" "#PWR019" (at 111.76 189.23 0)
+      (effects (font (size 1.27 1.27)) hide)
+    )
+    (property "Value" "GND" (at 111.76 187.96 0)
+      (effects (font (size 1.27 1.27)))
+    )
+    (property "Footprint" "" (at 111.76 182.88 0)
+      (effects (font (size 1.27 1.27)) hide)
+    )
+    (property "Datasheet" "" (at 111.76 182.88 0)
+      (effects (font (size 1.27 1.27)) hide)
+    )
+    (pin "1")
+    (instances
+      (project "Pi Hat"
+        (path "/2837f593-2859-4fb0-9481-b616afb06594"
+          (reference "#PWR019") (unit 1)
+        )
+      )
+    )
+  )
+  (symbol (lib_id "Connector_Generic:Conn_01x02") (at 256.54 40.64 0) (mirror x) (unit 1)
+    (in_bom yes) (on_board yes) (dnp no)
+    (property "Reference" "J4" (at 259.08 40.64 0)
       (effects (font (size 1.27 1.27)) (justify left))
     )
-    (property "Value" "Conn_01x02" (at 259.08 40.64 0)
+    (property "Value" "Conn_01x02" (at 259.08 38.1 0)
       (effects (font (size 1.27 1.27)) (justify left))
     )
-    (property "Footprint" "Connector_Molex:Molex_KK-254_AE-6410-02A_1x02_P2.54mm_Vertical" (at 256.54 38.1 0)
-      (effects (font (size 1.27 1.27)) hide)
-    )
-    (property "Datasheet" "~" (at 256.54 38.1 0)
+    (property "Footprint" "Connector_Molex:Molex_KK-254_AE-6410-02A_1x02_P2.54mm_Vertical" (at 256.54 40.64 0)
+      (effects (font (size 1.27 1.27)) hide)
+    )
+    (property "Datasheet" "~" (at 256.54 40.64 0)
       (effects (font (size 1.27 1.27)) hide)
     )
@@
         (path "/2837f593-2859-4fb0-9481-b616afb06594"
           (reference "R2") (unit 1)
+        )
+      )
+    )
+  )
+  (symbol (lib_id "Connector_Generic:Conn_01x03") (at 119.38 177.8 0) (unit 1)
+    (in_bom yes) (on_board yes) (dnp no) (fields_autoplaced)
+    (property "Reference" "J5" (at 121.92 176.53 0)
+      (effects (font (size 1.27 1.27)) (justify left))
+    )
+    (property "Value" "Conn_01x03" (at 121.92 179.07 0)
+      (effects (font (size 1.27 1.27)) (justify left))
+    )
+    (property "Footprint" "Connector_Molex:Molex_KK-254_AE-6410-03A_1x03_P2.54mm_Vertical" (at 119.38 177.8 0)
+      (effects (font (size 1.27 1.27)) hide)
+    )
+    (property "Datasheet" "~" (at 119.38 177.8 0)
+      (effects (font (size 1.27 1.27)) hide)
+    )
+    (pin "1")
+    (pin "3")
+    (pin "2")
+    (instances
+      (project "Pi Hat"
+        (path "/2837f593-2859-4fb0-9481-b616afb06594"
+          (reference "J5") (unit 1)
         )
       )
@@
         )
       )
+    )
+  )
+  (symbol (lib_id "power:+5V") (at 111.76 172.72 0) (mirror y) (unit 1)
+    (in_bom yes) (on_board yes) (dnp no)
+    (property "Reference" "#PWR018" (at 111.76 176.53 0)
+      (effects (font (size 1.27 1.27)) hide)
+    )
+    (property "Value" "+5V" (at 111.76 167.64 0)
+      (effects (font (size 1.27 1.27)))
+    )
+    (property "Footprint" "" (at 111.76 172.72 0)
+      (effects (font (size 1.27 1.27)) hide)
+    )
+    (property "Datasheet" "" (at 111.76 172.72 0)
+      (effects (font (size 1.27 1.27)) hide)
+    )
+    (pin "1")
+    (instances
+      (project "Pi Hat"
+        (path "/2837f593-2859-4fb0-9481-b616afb06594"
+          (reference "#PWR018") (unit 1)
+        )
+      )
